Commit message: Updated :robot:

File: kuka_description/urdf/kr4r600_macro.urdf.xacro (robot description, xacro)
@@ -1,8 +1,8 @@
 <?xml version="1.0"?>
 <robot xmlns:xacro="http://wiki.ros.org/xacro">
+  <xacro:include filename="$(find kuka_resources)/urdf/common_materials.xacro"/>
+  <xacro:include filename="$(find kuka_description)/urdf/kuka.transmission.xacro" />
   <xacro:include filename="$(find kuka_description)/urdf/kuka.gazebo.xacro" />
-  <xacro:include filename="$(find kuka_description)/urdf/common.gazebo.xacro" />
-  <xacro:include filename="$(find kuka_resources)/urdf/common_materials.xacro"/>
-  <xacro:macro name="kuka_kr4r600" params="prefix">
+  <xacro:macro name="kuka_kr4r600" params="prefix transmission_hw_interface:=hardware_interface/PositionJointInterface">
     <link name="${prefix}base_link">
       <visual>
@@ -215,4 +215,6 @@
       <origin xyz="0 0 0" rpy="0 ${radians(90)} 0"/>
     </joint>
+  <xacro:kuka_arm_transmission prefix="${prefix}" hw_interface="${transmission_hw_interface}" />
+  <xacro:kuka_arm_gazebo prefix="${prefix}" />
     <!-- ROS base_link to KUKA $ROBROOT coordinate system transform -->
     <link name="${prefix}base" />

File: kuka_description/urdf/kuka.gazebo.xacro (robot description, xacro)
@@ -1,5 +1,5 @@
 <?xml version="1.0"?>
 <robot xmlns:xacro="http://wiki.ros.org/xacro">
-  <xacro:macro name="kuka_kr4r600_gazebo" params="prefix">
+  <xacro:macro name="kuka_arm_gazebo" params="prefix">
     <gazebo reference="${prefix}joint_a1">
       <selfCollide>true</selfCollide>

File: kuka_description/urdf/training_table.urdf.xacro (robot description, xacro)
@@ -3,7 +3,14 @@
 <robot xmlns:xacro="http://ros.org/wiki/xacro"
        name="kuka_kr4r600" >
+  <xacro:arg name="transmission_hw_interface" default="hardware_interface/PositionJointInterface"/>
+  <xacro:include filename="$(find kuka_description)/urdf/common.gazebo.xacro" />
   <!-- kuka_kr4r600 robot arm -->
   <xacro:include filename="$(find kuka_description)/urdf/kr4r600_macro.urdf.xacro"/>
-  <xacro:kuka_kr4r600 prefix="" />
+<!-- legal values:
+     - hardware_interface/PositionJointInterface
+     - hardware_interface/VelocityJointInterface
+     - hardware_interface/EffortJointInterface
+-->
+  <xacro:kuka_kr4r600 prefix="" transmission_hw_interface="$(arg transmission_hw_interface)"/>
   <link name="world" />
   <xacro:include filename="$(find kuka_description)/urdf/table.urdf.xacro"/>
