Commit message: New files for model description

File: kuka_description/urdf/common.gazebo.xacro (robot description, xacro)
@@ -2,5 +2,8 @@
 <robot xmlns:xacro="http://ros.org/wiki/xacro">
   <gazebo>
-    <plugin name="ros_control" filename="libgazebo_ros_control.so"/>
+    <plugin name="ros_control" filename="libgazebo_ros_control.so">
+      <robotNamespace>/</robotNamespace>
+      <robotSimType>gazebo_ros_control/DefaultRobotHWSim</robotSimType>
+    </plugin>
   </gazebo>
 </robot>

File: kuka_description/urdf/kr4r600_macro.xacro (robot description, xacro)
@@ -1,10 +1,21 @@
 <?xml version="1.0"?>
 <robot xmlns:xacro="http://wiki.ros.org/xacro">
+    <xacro:macro name="default_inertial" params="mass">
+        <inertial>
+            <mass value="${mass}" />
+            <inertia ixx="1.0" ixy="0.0" ixz="0.0"
+                iyy="1.0" iyz="0.0"
+                izz="1.0" />
+        </inertial>
+    </xacro:macro>
   <xacro:include filename="$(find kuka_resources)/urdf/common_materials.xacro"/>
-  <xacro:include filename="$(find kuka_description)/urdf/kuka.transmission.xacro" />
-  <xacro:include filename="$(find kuka_description)/urdf/kuka.gazebo.xacro" />
+  <!-- <xacro:include filename="$(find kuka_description)/urdf/kuka.transmission.xacro" /> -->
+  <!-- <xacro:include filename="$(find kuka_description)/urdf/kuka.gazebo.xacro" /> -->
 <!--
   <xacro:macro name="kuka_kr4r600" params="prefix transmission_hw_interface:=hardware_interface/EffortJointInterface"> -->
+  <xacro:include filename="$(find kuka_resources)/urdf/common_constants.xacro"/>
+  <xacro:macro name="kuka_kr4r600" params="prefix">
     <link name="${prefix}base_link">
+    <xacro:default_inertial mass="1"/>
       <visual>
         <origin xyz="0 0 0" rpy="0 0 0" />
@@ -20,4 +31,5 @@
         </geometry>
       </collision>
+<!--
       <inertial>
         <origin xyz="0 0 0" rpy="0 0 0"/>
@@ -27,7 +39,8 @@
             iyy="49449443328.00000" iyz="74363816.000000"
             izz="47570612224.000000"/>
-      </inertial>
+      </inertial> -->
     </link>
     <link name="${prefix}link_1">
+    <xacro:default_inertial mass="1"/>
       <visual>
         <origin xyz="0 0 0" rpy="0 0 0" />
@@ -43,4 +56,5 @@
         </geometry>
       </collision>
+<!--
       <inertial>
         <origin xyz="0 0 0" rpy="0 0 0"/>
@@ -50,7 +64,8 @@
           iyy="18764271616.000000" iyz="180538688.000000"
           izz="20780234752.000000"/>
-      </inertial>
+      </inertial> -->
     </link>
     <link name="${prefix}link_2">
+    <xacro:default_inertial mass="1"/>
       <visual>
         <origin xyz="0 0 0" rpy="0 0 0" />
@@ -66,4 +81,5 @@
         </geometry>
       </collision>
+<!--
       <inertial>
         <origin xyz="0 0 0" rpy="0 0 0"/>
@@ -74,6 +90,8 @@
           izz="62598627328.000000"/>
       </inertial>
+ -->
     </link>
     <link name="${prefix}link_3">
+    <xacro:default_inertial mass="1"/>
       <visual>
         <origin xyz="0 0 0" rpy="0 0 0" />
@@ -89,4 +107,5 @@
         </geometry>
       </collision>
+<!--
       <inertial>
         <origin xyz="0 0 0" rpy="0 0 0"/>
@@ -96,7 +115,8 @@
           iyy="10409157632.000000" iyz="13806910.000000"
           izz="10024766464.000000"/>
-      </inertial>
+      </inertial> -->
     </link>
     <link name="${prefix}link_4">
+    <xacro:default_inertial mass="1"/>
       <visual>
         <origin xyz="0 0 0" rpy="0 0 0" />
@@ -112,4 +132,5 @@
         </geometry>
       </collision>
+<!--
       <inertial>
         <origin xyz="0 0 0" rpy="0 0 0"/>
@@ -119,7 +140,8 @@
           iyy="2560956160.000000" iyz="-46212612.000000"
           izz="3653170944.000000"/>
-      </inertial>
+      </inertial> -->
     </link>
     <link name="${prefix}link_5">
+    <xacro:default_inertial mass="1"/>
       <visual>
         <origin xyz="0 0 0" rpy="0 0 0" />
@@ -135,4 +157,5 @@
         </geometry>
       </collision>
+<!--
       <inertial>
         <origin xyz="0 0 0" rpy="0 0 0"/>
@@ -142,7 +165,8 @@
           iyy=" 642145344.000000" iyz="98441.296875"
           izz="684424448.000000"/>
-      </inertial>
+      </inertial> -->
     </link>
     <link name="${prefix}link_6">
+    <xacro:default_inertial mass="1"/>
       <visual>
         <origin xyz="0 0 0" rpy="0 0 0" />
@@ -158,4 +182,5 @@
         </geometry>
       </collision>
+<!--
       <inertial>
         <origin xyz="0 0 0" rpy="0 0 0"/>
@@ -165,5 +190,5 @@
           iyy=" 6104710.000000" iyz="2659.174805"
           izz="6102781.000000"/>
-      </inertial>
+      </inertial> -->
     </link>
     <!-- This frame corresponds to the $FLANGE coordinate system in KUKA KRC controllers. -->
@@ -174,5 +199,5 @@
       <child link="${prefix}link_1"/>
       <axis xyz="0 0 -1"/>
-      <limit lower="${radians(-170)}" upper="${radians(170)}" effort="0" velocity="${radians(530)}"/>
+      <limit lower="${-DEG2RAD * 170}" upper="${DEG2RAD * 170}" effort="100" velocity="${DEG2RAD* 530}"/>
     </joint>
     <joint name="${prefix}joint_a2" type="revolute">
@@ -181,5 +206,5 @@
       <child link="${prefix}link_2"/>
       <axis xyz="0 1 0"/>
-      <limit lower="${radians(-195)}" upper="${radians(40)}" effort="0" velocity="${radians(529)}"/>
+      <limit lower="${-DEG2RAD * 195}" upper="${DEG2RAD * 40}" effort="100" velocity="${DEG2RAD *529}"/>
     </joint>
     <joint name="${prefix}joint_a3" type="revolute">
@@ -188,5 +213,5 @@
       <child link="${prefix}link_3"/>
       <axis xyz="0 1 0"/>
-      <limit lower="${radians(-115)}" upper="${radians(150)}" effort="0" velocity="${radians(538)}"/>
+      <limit lower="${-DEG2RAD * 115}" upper="${DEG2RAD * 150}" effort="100" velocity="${DEG2RAD * 538}"/>
     </joint>
     <joint name="${prefix}joint_a4" type="revolute">
@@ -195,5 +220,5 @@
       <child link="${prefix}link_4"/>
       <axis xyz="-1 0 0"/>
-      <limit lower="${radians(-185)}" upper="${radians(185)}" effort="0" velocity="${radians(600)}"/>
+      <limit lower="${-DEG2RAD * 185}" upper="${DEG2RAD * 185}" effort="100" velocity="${DEG2RAD * 600}"/>
     </joint>
     <joint name="${prefix}joint_a5" type="revolute">
@@ -202,5 +227,5 @@
       <child link="${prefix}link_5"/>
       <axis xyz="0 1 0"/>
-      <limit lower="${radians(-120)}" upper="${radians(120)}" effort="0" velocity="${radians(600)}"/>
+      <limit lower="${-DEG2RAD * 120}" upper="${DEG2RAD * 120}" effort="100" velocity="${DEG2RAD * 600}"/>
     </joint>
     <joint name="${prefix}joint_a6" type="revolute">
@@ -209,13 +234,14 @@
       <child link="${prefix}link_6"/>
       <axis xyz="-1 0 0"/>
-      <limit lower="${radians(-350)}" upper="${radians(350)}" effort="0" velocity="${radians(800)}"/>
+      <limit lower="${-DEG2RAD * 350}" upper="${DEG2RAD* 350}" effort="100" velocity="${DEG2RAD* 800}"/>
     </joint>
     <joint name="${prefix}joint_a6-tool0" type="fixed">
       <parent link="${prefix}link_6"/>
       <child link="${prefix}tool0"/>
-      <origin xyz="0 0 0" rpy="0 ${radians(90)} 0"/>
-    </joint>
-  <xacro:kuka_arm_transmission prefix="${prefix}" hw_interface="${transmission_hw_interface}" />
+      <origin xyz="0 0 0" rpy="0 ${DEG2RAD * 90} 0"/>
+    </joint>
+<!--   <xacro:kuka_arm_transmission prefix="${prefix}" hw_interface="${transmission_hw_interface}" />
   <xacro:kuka_arm_gazebo prefix="${prefix}" />
+ -->
     <!-- ROS base_link to KUKA $ROBROOT coordinate system transform -->
     <link name="${prefix}base" />

File: kuka_description/urdf/kuka.transmission.xacro (robot description, xacro)
@@ -1,9 +1,10 @@
 <?xml version="1.0"?>
 <robot xmlns:xacro="http://ros.org/wiki/xacro">
-  <xacro:macro name="kuka_arm_transmission" params="prefix hw_interface">
+  <xacro:macro name="kuka_arm_transmission" params="prefix">
+    <xacro:kuka_kr4r600 prefix="${prefix}" />
     <transmission name="${prefix}joint_a1_trans">
       <type>transmission_interface/SimpleTransmission</type>
       <joint name="${prefix}joint_a1">
-        <hardwareInterface>${hw_interface}</hardwareInterface>
+        <hardwareInterface>hardware_interface/EffortJointInterface</hardwareInterface>
       </joint>
       <actuator name="${prefix}joint_a1_motor">
@@ -14,5 +15,5 @@
       <type>transmission_interface/SimpleTransmission</type>
       <joint name="${prefix}joint_a2">
-        <hardwareInterface>${hw_interface}</hardwareInterface>
+        <hardwareInterface>hardware_interface/EffortJointInterface</hardwareInterface>
       </joint>
       <actuator name="${prefix}joint_a2_motor">
@@ -23,5 +24,5 @@
       <type>transmission_interface/SimpleTransmission</type>
       <joint name="${prefix}joint_a3">
-        <hardwareInterface>${hw_interface}</hardwareInterface>
+        <hardwareInterface>hardware_interface/EffortJointInterface</hardwareInterface>
       </joint>
       <actuator name="${prefix}joint_a3_motor">
@@ -32,7 +33,7 @@
       <type>transmission_interface/SimpleTransmission</type>
       <joint name="${prefix}joint_a4">
-        <hardwareInterface>${hw_interface}</hardwareInterface>
+        <hardwareInterface>hardware_interface/EffortJointInterface</hardwareInterface>
       </joint>
-      <actuator name="$joint_a4_motor">
+      <actuator name="${prefix}joint_a4_motor">
         <mechanicalReduction>1</mechanicalReduction>
       </actuator>
@@ -41,5 +42,5 @@
       <type>transmission_interface/SimpleTransmission</type>
       <joint name="${prefix}joint_a5">
-        <hardwareInterface>${hw_interface}</hardwareInterface>
+        <hardwareInterface>hardware_interface/EffortJointInterface</hardwareInterface>
       </joint>
       <actuator name="${prefix}joint_a5_motor">
@@ -50,5 +51,5 @@
       <type>transmission_interface/SimpleTransmission</type>
       <joint name="${prefix}joint_a6">
-        <hardwareInterface>${hw_interface}</hardwareInterface>
+        <hardwareInterface>hardware_interface/EffortJointInterface</hardwareInterface>
       </joint>
       <actuator name="${prefix}joint_a6_motor">

File: kuka_description/urdf/training_table.urdf.xacro (robot description, xacro)
@@ -1,10 +1,9 @@
 <?xml version="1.0"?>
 <!-- <robot name="kuka_kr4r600" xmlns:xacro="http://wiki.ros.org/xacro"> -->
-<robot xmlns:xacro="http://ros.org/wiki/xacro"
-       name="kuka_kr4r600" >
-  <xacro:arg name="transmission_hw_interface" default="hardware_interface/PositionJointInterface"/>
-  <xacro:include filename="$(find kuka_description)/urdf/common.gazebo.xacro" />
+<robot xmlns:xacro="http://ros.org/wiki/xacro" name="kuka_kr4r600" >
+  <!-- <xacro:arg name="transmission_hw_interface" default="hardware_interface/PositionJointInterface"/> -->
+  <!-- <xacro:include filename="$(find kuka_description)/urdf/common.gazebo.xacro" /> -->
   <!-- kuka_kr4r600 robot arm -->
-  <xacro:include filename="$(find kuka_description)/urdf/kr4r600_macro.urdf.xacro"/>
+  <xacro:include filename="$(find kuka_description)/urdf/kuka_kr4r600_macro.xacro"/>
 <!-- legal values:
      - hardware_interface/PositionJointInterface
@@ -12,5 +11,5 @@
      - hardware_interface/EffortJointInterface
 -->
-  <xacro:kuka_kr4r600 prefix="" transmission_hw_interface="$(arg transmission_hw_interface)"/>
+  <xacro:kuka_kr4r600_gazebo prefix="" />
   <link name="world" />
   <xacro:include filename="$(find kuka_description)/urdf/table.urdf.xacro"/>
