Commit message: Added gazebo camera

File: kuka_description/urdf/kr4r600_macro.xacro (robot description, xacro)
@@ -10,4 +10,5 @@
     </xacro:macro>
   <xacro:include filename="$(find kuka_resources)/urdf/common_materials.xacro"/>
+  <xacro:property name="camera_link" value="0.05" /> <!-- Size of square 'camera' box -->
   <!-- <xacro:include filename="$(find kuka_description)/urdf/kuka.transmission.xacro" /> -->
   <!-- <xacro:include filename="$(find kuka_description)/urdf/kuka.gazebo.xacro" /> -->
@@ -31,5 +32,4 @@
         </geometry>
       </collision>
-<!--
       <inertial>
         <origin xyz="0 0 0" rpy="0 0 0"/>
@@ -39,5 +39,5 @@
             iyy="49449443328.00000" iyz="74363816.000000"
             izz="47570612224.000000"/>
-      </inertial> -->
+      </inertial>
     </link>
     <link name="${prefix}link_1">
@@ -56,5 +56,4 @@
         </geometry>
       </collision>
-<!--
       <inertial>
         <origin xyz="0 0 0" rpy="0 0 0"/>
@@ -64,5 +63,5 @@
           iyy="18764271616.000000" iyz="180538688.000000"
           izz="20780234752.000000"/>
-      </inertial> -->
+      </inertial>
     </link>
     <link name="${prefix}link_2">
@@ -81,5 +80,4 @@
         </geometry>
       </collision>
-<!--
       <inertial>
         <origin xyz="0 0 0" rpy="0 0 0"/>
@@ -90,5 +88,4 @@
           izz="62598627328.000000"/>
       </inertial>
- -->
     </link>
     <link name="${prefix}link_3">
@@ -107,5 +104,4 @@
         </geometry>
       </collision>
-<!--
       <inertial>
         <origin xyz="0 0 0" rpy="0 0 0"/>
@@ -115,5 +111,5 @@
           iyy="10409157632.000000" iyz="13806910.000000"
           izz="10024766464.000000"/>
-      </inertial> -->
+      </inertial>
     </link>
     <link name="${prefix}link_4">
@@ -132,5 +128,4 @@
         </geometry>
       </collision>
-<!--
       <inertial>
         <origin xyz="0 0 0" rpy="0 0 0"/>
@@ -140,5 +135,5 @@
           iyy="2560956160.000000" iyz="-46212612.000000"
           izz="3653170944.000000"/>
-      </inertial> -->
+      </inertial>
     </link>
     <link name="${prefix}link_5">
@@ -157,5 +152,4 @@
         </geometry>
       </collision>
-<!--
       <inertial>
         <origin xyz="0 0 0" rpy="0 0 0"/>
@@ -165,5 +159,5 @@
           iyy=" 642145344.000000" iyz="98441.296875"
           izz="684424448.000000"/>
-      </inertial> -->
+      </inertial>
     </link>
     <link name="${prefix}link_6">
@@ -182,5 +176,4 @@
         </geometry>
       </collision>
-<!--
       <inertial>
         <origin xyz="0 0 0" rpy="0 0 0"/>
@@ -190,8 +183,29 @@
           iyy=" 6104710.000000" iyz="2659.174805"
           izz="6102781.000000"/>
-      </inertial> -->
+      </inertial>
     </link>
     <!-- This frame corresponds to the $FLANGE coordinate system in KUKA KRC controllers. -->
     <link name="${prefix}tool0"/>
+  <!-- Camera -->
+    <link name="camera_link">
+      <collision>
+        <origin xyz="0 0 0" rpy="0 0 0"/>
+        <geometry>
+      <box size="${camera_link} ${camera_link} ${camera_link}"/>
+        </geometry>
+      </collision>
+      <visual>
+        <origin xyz="0 0 0" rpy="0 0 0"/>
+        <geometry>
+      <box size="${camera_link} ${camera_link} ${camera_link}"/>
+        </geometry>
+        <material name="red"/>
+      </visual>
+      <inertial>
+        <mass value="1e-5" />
+        <origin xyz="0 0 0" rpy="0 0 0"/>
+        <inertia ixx="1e-6" ixy="0" ixz="0" iyy="1e-6" iyz="0" izz="1e-6" />
+      </inertial>
+    </link>
     <joint name="${prefix}joint_a1" type="revolute">
       <origin xyz="0 0 0.33" rpy="0 0 0"/>
@@ -240,4 +254,10 @@
       <child link="${prefix}tool0"/>
       <origin xyz="0 0 0" rpy="0 ${DEG2RAD * 90} 0"/>
+    </joint>
+   <joint name="camera_joint" type="fixed">
+      <axis xyz="0 0 0" />
+      <origin xyz="0 0 0" rpy="0 30 0"/>
+      <parent link="${prefix}tool0"/>
+      <child link="camera_link"/>
     </joint>
 <!--   <xacro:kuka_arm_transmission prefix="${prefix}" hw_interface="${transmission_hw_interface}" />

File: kuka_description/urdf/kuka_kr4r600_macro.xacro (robot description, xacro)
@@ -97,4 +97,44 @@
     </plugin>
   </gazebo>
+ <!-- camera -->
+  <gazebo reference="camera_link">
+    <sensor type="camera" name="camera1">
+      <update_rate>30.0</update_rate>
+      <camera name="head">
+        <horizontal_fov>1.3962634</horizontal_fov>
+        <image>
+          <width>800</width>
+          <height>800</height>
+          <format>R8G8B8</format>
+        </image>
+        <clip>
+          <near>0.02</near>
+          <far>300</far>
+        </clip>
+        <noise>
+          <type>gaussian</type>
+          <!-- Noise is sampled independently per pixel on each frame.
+               That pixel's noise value is added to each of its color
+               channels, which at that point lie in the range [0,1]. -->
+          <mean>0.0</mean>
+          <stddev>0.007</stddev>
+        </noise>
+      </camera>
+      <plugin name="camera_controller" filename="libgazebo_ros_camera.so">
+        <alwaysOn>true</alwaysOn>
+        <updateRate>0.0</updateRate>
+        <cameraName>kuka/camera1</cameraName>
+        <imageTopicName>image_raw</imageTopicName>
+        <cameraInfoTopicName>camera_info</cameraInfoTopicName>
+        <frameName>camera_link</frameName>
+        <hackBaseline>0.07</hackBaseline>
+        <distortionK1>0.0</distortionK1>
+        <distortionK2>0.0</distortionK2>
+        <distortionK3>0.0</distortionK3>
+        <distortionT1>0.0</distortionT1>
+        <distortionT2>0.0</distortionT2>
+      </plugin>
+    </sensor>
+  </gazebo>
   </xacro:macro>
 </robot>

File: kuka_description/urdf/training_table.urdf.xacro (robot description, xacro)
@@ -20,6 +20,6 @@
     <origin xyz="0.0 0.0 0.0" rpy="0.0 0.0 0.0" />
   </joint>
-<!-- attach the robot to the box -->
-  <joint name="box_joint" type="fixed">
+<!-- attach the robot to the table -->
+  <joint name="table_joint" type="fixed">
     <parent link="table_top_link"/>
     <child link="base_link"/>

Commit message: Added transmission interface

File: kuka_description/urdf/kr4r600_macro.xacro (robot description, xacro)
@@ -13,8 +13,7 @@
   <!-- <xacro:include filename="$(find kuka_description)/urdf/kuka.transmission.xacro" /> -->
   <!-- <xacro:include filename="$(find kuka_description)/urdf/kuka.gazebo.xacro" /> -->
-<!--
-  <xacro:macro name="kuka_kr4r600" params="prefix transmission_hw_interface:=hardware_interface/EffortJointInterface"> -->
+  <xacro:macro name="kuka_kr4r600" params="prefix transmission_hw_interface:=hardware_interface/EffortJointInterface">
   <xacro:include filename="$(find kuka_resources)/urdf/common_constants.xacro"/>
-  <xacro:macro name="kuka_kr4r600" params="prefix">
+  <!-- <xacro:macro name="kuka_kr4r600" params="prefix"> -->
     <link name="${prefix}base_link">
     <xacro:default_inertial mass="1"/>

Commit message: Added hokuyo scan

File: kuka_description/urdf/kr4r600_macro.xacro (robot description, xacro)
@@ -191,13 +191,33 @@
         <origin xyz="0 0 0" rpy="0 0 0"/>
         <geometry>
-      <box size="${camera_link} ${camera_link} ${camera_link}"/>
-        </geometry>
-      </collision>
-      <visual>
-        <origin xyz="0 0 0" rpy="0 0 0"/>
-        <geometry>
-      <box size="${camera_link} ${camera_link} ${camera_link}"/>
-        </geometry>
-        <material name="red"/>
+          <box size="0.05 0.05 0.05"/>
+        </geometry>
+      </collision>
+      <visual>
+        <origin xyz="0 0 0" rpy="0 0 0"/>
+        <geometry>
+          <box size="0.05 0.05 0.05"/>
+        </geometry>
+        <material name="white"/>
+      </visual>
+      <inertial>
+        <mass value="1e-5" />
+        <origin xyz="0 0 0" rpy="0 0 0"/>
+        <inertia ixx="1e-6" ixy="0" ixz="0" iyy="1e-6" iyz="0" izz="1e-6" />
+      </inertial>
+    </link>
+    <!-- Hokuyo Laser -->
+    <link name="hokuyo_link">
+      <collision>
+        <origin xyz="0 0 0" rpy="0 0 0"/>
+        <geometry>
+          <box size="0.05 0.05 0.05"/>
+        </geometry>
+      </collision>
+      <visual>
+        <origin xyz="0 0 0" rpy="0 0 0"/>
+        <geometry>
+          <box size="0.05 0.05 0.05"/>
+        </geometry>
       </visual>
       <inertial>
@@ -254,9 +274,13 @@
       <origin xyz="0 0 0" rpy="0 ${DEG2RAD * 90} 0"/>
     </joint>
-   <joint name="camera_joint" type="fixed">
-      <axis xyz="0 0 0" />
-      <origin xyz="0 0 0" rpy="0 30 0"/>
+    <joint name="camera_joint" type="fixed">
+      <origin xyz="0 0 0.025" rpy="0 -1.5708 0"/>
       <parent link="${prefix}tool0"/>
       <child link="camera_link"/>
+    </joint>
+    <joint name="hokuyo_joint" type="fixed">
+      <origin xyz="0 0.05 0" rpy="0 0 0"/>
+      <parent link="camera_link"/>
+      <child link="hokuyo_link"/>
     </joint>
 <!--   <xacro:kuka_arm_transmission prefix="${prefix}" hw_interface="${transmission_hw_interface}" />
@@ -264,10 +288,10 @@
  -->
     <!-- ROS base_link to KUKA $ROBROOT coordinate system transform -->
-    <link name="${prefix}base" />
+<!--     <link name="${prefix}base" />
     <joint name="${prefix}base_link-base" type="fixed">
       <origin xyz="0 0 0" rpy="0 0 0"/>
       <parent link="${prefix}base_link"/>
       <child link="${prefix}base"/>
-    </joint>
+    </joint> -->
   </xacro:macro>
 </robot>

File: kuka_description/urdf/kuka_kr4r600_macro.xacro (robot description, xacro)
@@ -133,34 +133,8 @@
     </sensor>
   </gazebo>
-  <joint name="hokuyo_joint" type="fixed">
-      <axis xyz="0 0 0" />
-      <origin xyz="0 0.0 0.0" rpy="0 0 0"/>
-      <parent link="camera_link"/>
-      <child link="hokuyo_link"/>
-    </joint>
-    <!-- Hokuyo Laser -->
-    <link name="hokuyo_link">
-      <collision>
-        <origin xyz="0 0 0" rpy="0 0 0"/>
-        <geometry>
-          <box size="0.05 0.05 0.05"/>
-        </geometry>
-      </collision>
-      <visual>
-        <origin xyz="0 0 0" rpy="0 0 0"/>
-        <geometry>
-          <box size="0.05 0.05 0.05"/>
-        </geometry>
-      </visual>
-      <inertial>
-        <mass value="1e-5" />
-        <origin xyz="0 0 0" rpy="0 0 0"/>
-        <inertia ixx="1e-6" ixy="0" ixz="0" iyy="1e-6" iyz="0" izz="1e-6" />
-      </inertial>
-    </link>
  <!-- hokuyo -->
   <gazebo reference="hokuyo_link">
     <sensor type="gpu_ray" name="head_hokuyo_sensor">
-      <pose>0.5 0 0 0 0 0</pose>
+      <pose>0 0 0 0 0 0</pose>
       <visualize>false</visualize>
       <update_rate>40</update_rate>
