Commit message: Updated training table

File: kuka_description/urdf/training_table.urdf.xacro (robot description, xacro)
@@ -3,35 +3,20 @@
 <robot xmlns:xacro="http://ros.org/wiki/xacro"
        name="kuka_kr4r600" >
-  <!-- common stuff -->
-  <!-- <xacro:include filename="$(find ur_description)/urdf/common.gazebo.xacro" /> -->
-  <!-- ur3 -->
-  <!-- <xacro:include filename="$(find ur_description)/urdf/ur3.urdf.xacro" /> -->
+  <!-- kuka_kr4r600 robot arm -->
   <xacro:include filename="$(find kuka_kr4_support)/urdf/kr4r600_macro.xacro"/>
-  <!-- arm -->
   <xacro:kuka_kr4r600 prefix="" />
   <link name="world" />
-<!-- box-->
-  <link name="box_link">
-    <visual>
-      <geometry>
-        <box size="1.0 1.0 0.86"/>
-      </geometry>
-    </visual>
-  </link>
-<!-- attach the box to the world-->
+  <xacro:include filename="$(find kuka_description)/urdf/table.urdf.xacro"/>
+<!-- attach the table to the world-->
   <joint name="world_joint" type="fixed">
     <parent link="world" />
-    <child link = "box_link" />
-    <origin xyz="0.0 0.0 0.43" rpy="0.0 0.0 0.0" />
+    <child link = "table_top_link" />
+    <origin xyz="0.0 0.0 0.0" rpy="0.0 0.0 0.0" />
   </joint>
 <!-- attach the robot to the box -->
   <joint name="box_joint" type="fixed">
-    <parent link="box_link"/>
+    <parent link="table_top_link"/>
     <child link="base_link"/>
-    <origin xyz="0.0 0.0 0.43" rpy="0 0 1.57" />
+    <origin xyz="1.0 0.0 0.8" rpy="0 0 0" />
   </joint>
-<!--astra  -->
-<!-- <xacro:include filename="$(find manos_description)/urdf/sensors/kinect.urdf.xacro"/> -->
-<!--attach the kinect to the robot -->
- <!-- <xacro:sensor_kinect  parent="base_link"/> -->
 </robot>

Commit message: Changed table origin

File: kuka_description/urdf/training_table.urdf.xacro (robot description, xacro)
@@ -24,5 +24,23 @@
     <parent link="table_top_link"/>
     <child link="base_link"/>
-    <origin xyz="1.0 0.0 0.8" rpy="0 0 0" />
+    <origin xyz="0 0.0 0.8" rpy="0 0 0" />
+  </joint>
+<!--Add box to the table-->
+  <link name="box_link">
+    <visual>
+      <geometry>
+        <box size="0.10 0.10 0.10"/>
+      </geometry>
+    </visual>
+  </link>
+  <gazebo reference="box_link">
+    <material>Gazebo/Red</material>
+    <turnGravityOff>true</turnGravityOff>
+  </gazebo>
+  <!-- attach the box to the table-->
+  <joint name="box_joint" type="fixed">
+    <parent link="table_top_link" />
+    <child link = "box_link" />
+    <origin xyz="0.5 0.0 0.85" rpy="0.0 0.0 0.0" />
   </joint>
 </robot>

Commit message: Changed position of base_link

File: kuka_description/urdf/training_table.urdf.xacro (robot description, xacro)
@@ -17,12 +17,12 @@
   <joint name="world_joint" type="fixed">
     <parent link="world" />
-    <child link = "table_top_link" />
-    <origin xyz="0.0 0.0 0.0" rpy="0.0 0.0 0.0" />
+    <child link = "base_link" />
+    <origin xyz="0.0 0.0 0.8" rpy="0.0 0.0 0.0" />
   </joint>
 <!-- attach the robot to the table -->
   <joint name="table_joint" type="fixed">
-    <parent link="table_top_link"/>
-    <child link="base_link"/>
-    <origin xyz="0 0.0 0.8" rpy="0 0 0" />
+    <parent link="base_link"/>
+    <child link="table_top_link"/>
+    <origin xyz="0 0.0 -0.8" rpy="0 0 0" />
   </joint>
 <!--Add box to the table-->
@@ -33,8 +33,17 @@
       </geometry>
     </visual>
+    <collision>
+      <origin xyz ="0 0 0" rpy="0 0 0"/>
+      <geometry>
+        <box size="0.10 0.10 0.10"/>
+      </geometry>
+    </collision>
   </link>
   <gazebo reference="box_link">
     <material>Gazebo/Red</material>
-    <turnGravityOff>true</turnGravityOff>
+    <mu1>50.0</mu1>
+    <mu2>50.0</mu2>
+    <kp>1000000.0</kp>
+    <kd>1.0</kd>
   </gazebo>
   <!-- attach the box to the table-->

Commit message: Changed tables origin

File: kuka_description/urdf/training_table.urdf.xacro (robot description, xacro)
@@ -49,7 +49,7 @@
   <!-- attach the box to the table-->
   <joint name="box_joint" type="fixed">
-    <parent link="table_top_link" />
+    <parent link="base_link" />
     <child link = "box_link" />
-    <origin xyz="0.5 0.0 0.85" rpy="0.0 0.0 0.0" />
+    <origin xyz="0.5 0.0 0.05" rpy="0.0 0.0 0.0" />
   </joint>
 </robot>
