Commit message: Changed to rotonda table

File: kuka_description/urdf/table.urdf.xacro (robot description, xacro)
@@ -14,4 +14,5 @@
        xmlns:physics="http://playerstage.sourceforge.net/gazebo/xmlschema/#physics">
   <property name="table_height" value="0.8" />
+  <property name="table_radius" value="0.6" />
   <property name="table_width" value="1.2" />
   <property name="table_depth" value="1.2" />
@@ -34,5 +35,6 @@
       <origin xyz="${table_x} ${table_y} ${table_z+table_height-table_top_thickness/2}" />
       <geometry>
-        <box size="${table_width} ${table_depth} ${table_top_thickness}" />
+        <!-- <box size="${table_width} ${table_depth} ${table_top_thickness}" /> -->
+        <cylinder length="${table_top_thickness}" radius="${table_radius}"/>
       </geometry>
     </visual>
@@ -40,5 +42,6 @@
       <origin xyz="${table_x} ${table_y} ${table_z+table_height-table_top_thickness/2}" />
       <geometry>
-        <box size="${table_width} ${table_depth} ${table_top_thickness}" />
+        <cylinder length="${table_top_thickness}" radius="${table_radius}"/>
+        <!-- <box size="${table_width} ${table_depth} ${table_top_thickness}" /> -->
       </geometry>
     </collision>
@@ -53,5 +56,5 @@
   <joint name="leg1_joint" type="fixed" >
     <parent link="table_top_link" />
-    <origin xyz="${table_x+table_width/2} ${table_y+table_depth/2} ${table_z+table_height}" rpy="0 0 0" />
+    <origin xyz="${table_x+table_radius/2} ${table_y+table_radius/2} ${table_z+table_height }" rpy="0 0 0" />
     <child link="leg1_link" />
   </joint>
@@ -78,5 +81,5 @@
   </link>
   <gazebo reference="leg1_link">
-    <material>Gazebo/Red</material>
+    <material>Gazebo/White</material>
     <mu1>1000.0</mu1>
     <mu2>1000.0</mu2>
@@ -87,5 +90,5 @@
   <joint name="leg2_joint" type="fixed" >
     <parent link="table_top_link" />
-    <origin xyz="${table_x-table_width/2} ${table_y+table_depth/2} ${table_z+table_height}" rpy="0 0 0" />
+    <origin xyz="${table_x-table_radius/2} ${table_y+table_radius/2} ${table_z+table_height }" rpy="0 0 0" />
     <child link="leg2_link" />
   </joint>
@@ -112,5 +115,5 @@
   </link>
   <gazebo reference="leg2_link">
-    <material>Gazebo/Red</material>
+    <material>Gazebo/White</material>
     <mu1>1000.0</mu1>
     <mu2>1000.0</mu2>
@@ -121,5 +124,5 @@
   <joint name="leg3_joint" type="fixed" >
     <parent link="table_top_link" />
-    <origin xyz="${table_x+table_width/2} ${table_y-table_depth/2} ${table_z+table_height}" rpy="0 0 0" />
+    <origin xyz="${table_x+table_radius/2} ${table_y-table_radius/2} ${table_z+table_height}" rpy="0 0 0" />
     <child link="leg3_link" />
   </joint>
@@ -146,5 +149,5 @@
   </link>
   <gazebo reference="leg3_link">
-    <material>Gazebo/Red</material>
+    <material>Gazebo/White</material>
     <mu1>1000.0</mu1>
     <mu2>1000.0</mu2>
@@ -155,5 +158,5 @@
   <joint name="leg4_joint" type="fixed" >
     <parent link="table_top_link" />
-    <origin xyz="${table_x-table_width/2} ${table_y-table_depth/2} ${table_z+table_height}" rpy="0 0 0" />
+    <origin xyz="${table_x-table_radius/2} ${table_y-table_radius/2} ${table_z+table_height }" rpy="0 0 0" />
     <child link="leg4_link" />
   </joint>
@@ -180,5 +183,5 @@
   </link>
   <gazebo reference="leg4_link">
-    <material>Gazebo/Red</material>
+    <material>Gazebo/White</material>
     <mu1>1000.0</mu1>
     <mu2>1000.0</mu2>

Commit message: fixed for noetic

File: kuka_description/urdf/table.urdf.xacro (robot description, xacro)
@@ -2,4 +2,5 @@
 <robot name="table"
        xmlns:xi="http://www.w3.org/2001/XInclude"
+       xmlns:xacro="http://www.ros.org/wiki/xacro"
        xmlns:gazebo="http://playerstage.sourceforge.net/gazebo/xmlschema/#gz"
        xmlns:model="http://playerstage.sourceforge.net/gazebo/xmlschema/#model"
@@ -13,14 +14,14 @@
        xmlns:controller="http://playerstage.sourceforge.net/gazebo/xmlschema/#controller"
        xmlns:physics="http://playerstage.sourceforge.net/gazebo/xmlschema/#physics">
-  <property name="table_height" value="0.8" />
-  <property name="table_radius" value="0.6" />
-  <property name="table_width" value="1.2" />
-  <property name="table_depth" value="1.2" />
-  <property name="leg_radius" value="0.02" />
-  <property name="table_x" value="0.0" />
-  <property name="table_y" value="0.0" />
-  <property name="table_z" value="0.0" />
-  <property name="table_top_thickness" value="0.05"/>
-  <property name="M_PI" value="3.1415926535897931" />
+  <xacro:property name="table_height" value="0.8" />
+  <xacro:property name="table_radius" value="0.6" />
+  <xacro:property name="table_width" value="1.2" />
+  <xacro:property name="table_depth" value="1.2" />
+  <xacro:property name="leg_radius" value="0.02" />
+  <xacro:property name="table_x" value="0.0" />
+  <xacro:property name="table_y" value="0.0" />
+  <xacro:property name="table_z" value="0.0" />
+  <xacro:property name="table_top_thickness" value="0.05"/>
+  <xacro:property name="M_PI" value="3.1415926535897931" />
   <!-- tabletop height is .55+.01+.025=.585 -->
   <link name="table_top_link">
